File: SSTdriver.sch (KiCad schematic (older format))
At the start: 63 parts, among them P1 CONN_01X05, P2 USB_OTG, P3 CONN_01X04, Q1 Fairchild_BCV27, Q2 QRE1113, Q3 DMG3415U-7, Q4 DMG3415U-7, U1 ATMEGA328P-A, U2 FT231X, U3 LMV358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

Commit message: Fixed a trace clearance by usb interface chip.
Parts:
- C15, C19: footprint Capacitors_SMD:c_elec_8x10 -> Capacitors_SMD:CP_Elec_6.3x5.8
- U3: symbol LMV358 -> LMV358-RESCUE-SSTdriver
Changed lines of the file:
@@
 Sheet 1 1
 Title "Tracker Controller and Driver"
-Date "2016-12-24"
-Rev "2.1.0"
+Date "2017-05-31"
+Rev "2.1.1"
 Comp "StarSync Trackers LLC"
 Comment1 ""
@@
 F 0 "C15" H 8475 1200 50  0000 L CNN
 F 1 "47u" H 8475 1000 50  0000 L CNN
-F 2 "Capacitors_SMD:c_elec_8x10" H 8488 950 50  0001 C CNN
+F 2 "Capacitors_SMD:CP_Elec_6.3x5.8" H 8488 950 50  0001 C CNN
 F 3 "" H 8450 1100 50  0000 C CNN
 	1    8450 1100
@@
 F 0 "C19" H 9825 1200 50  0000 L CNN
 F 1 "47u" H 9825 1000 50  0000 L CNN
-F 2 "Capacitors_SMD:c_elec_8x10" H 9838 950 50  0001 C CNN
+F 2 "Capacitors_SMD:CP_Elec_6.3x5.8" H 9838 950 50  0001 C CNN
 F 3 "" H 9800 1100 50  0000 C CNN
 	1    9800 1100
@@
 Connection ~ 10050 850
 $Comp
-L LMV358 U3
+L LMV358-RESCUE-SSTdriver U3
 U 1 1 58560F68
 P 6850 2900
@@
 $EndComp
 $Comp
-L LMV358 U3
+L LMV358-RESCUE-SSTdriver U3
 U 2 1 58561005
 P 5000 2500
@@
 DTR
 $Comp
-L ATMEGA328P-A U1
-U 1 1 5856A373
-P 2150 5100
-F 0 "U1" H 1400 6350 50  0000 L BNN
-F 1 "ATMEGA328P-A" H 2550 3700 50  0000 L BNN
-F 2 "Housings_QFP:TQFP-32_7x7mm_Pitch0.8mm" H 2150 5100 50  0001 C CIN
-F 3 "" H 2150 5100 50  0000 C CNN
-	1    2150 5100
-	1    0    0    -1
-$EndComp
-$Comp
 L C C10
 U 1 1 5856A6A1
@@
 Connection ~ 1150 4000
 Wire Wire Line
-	1050 3950 1050 4000
+	1050 4000 1050 3950
 Connection ~ 1050 4000
 $Comp
@@
 	1050 3600 1050 3650
 $Comp
-L GND #PWR029
-U 1 1 5856C297
-P 1100 6200
-F 0 "#PWR029" H 1100 5950 50  0001 C CNN
-F 1 "GND" H 1100 6050 50  0000 C CNN
-F 2 "" H 1100 6200 50  0000 C CNN
-F 3 "" H 1100 6200 50  0000 C CNN
-	1    1100 6200
-	0    1    1    0
-$EndComp
-Wire Wire Line
-	1250 6100 1200 6100
-Wire Wire Line
-	1200 6100 1200 6300
-Wire Wire Line
-	1200 6300 1250 6300
-Wire Wire Line
-	1100 6200 1250 6200
-Connection ~ 1200 6200
-$Comp
 L CONN_01X05 P1
 U 1 1 5856D308
@@
 $EndComp
 $Comp
-L GND #PWR030
+L GND #PWR029
 U 1 1 5856DEEA
 P 5500 5450
-F 0 "#PWR030" H 5500 5200 50  0001 C CNN
+F 0 "#PWR029" H 5500 5200 50  0001 C CNN
 F 1 "GND" H 5500 5300 50  0000 C CNN
 F 2 "" H 5500 5450 50  0000 C CNN
@@
 Connection ~ 4450 5450
 $Comp
-L +5V #PWR031
+L +5V #PWR030
 U 1 1 5856EA42
 P 4200 5000
-F 0 "#PWR031" H 4200 4850 50  0001 C CNN
+F 0 "#PWR030" H 4200 4850 50  0001 C CNN
 F 1 "+5V" H 4200 5140 50  0000 C CNN
 F 2 "" H 4200 5000 50  0000 C CNN
@@
 	1050 7400 950  7400
 $Comp
-L GND #PWR032
+L GND #PWR031
 U 1 1 58571AF9
 P 1000 7550
-F 0 "#PWR032" H 1000 7300 50  0001 C CNN
+F 0 "#PWR031" H 1000 7300 50  0001 C CNN
 F 1 "GND" H 1000 7400 50  0000 C CNN
 F 2 "" H 1000 7550 50  0000 C CNN
@@
 	7750 4550 7850 4550
 $Comp
-L +5V #PWR033
+L +5V #PWR032
 U 1 1 5857722B
 P 7300 4200
-F 0 "#PWR033" H 7300 4050 50  0001 C CNN
+F 0 "#PWR032" H 7300 4050 50  0001 C CNN
 F 1 "+5V" H 7300 4340 50  0000 C CNN
 F 2 "" H 7300 4200 50  0000 C CNN
@@
 $EndComp
 $Comp
-L GND #PWR034
+L GND #PWR033
 U 1 1 58577408
 P 6850 4250
-F 0 "#PWR034" H 6850 4000 50  0001 C CNN
+F 0 "#PWR033" H 6850 4000 50  0001 C CNN
 F 1 "GND" H 6850 4100 50  0000 C CNN
 F 2 "" H 6850 4250 50  0000 C CNN
@@
 	9800 5100 9700 5100
 $Comp
-L GND #PWR035
+L GND #PWR034
 U 1 1 58579701
 P 9850 5050
-F 0 "#PWR035" H 9850 4800 50  0001 C CNN
+F 0 "#PWR034" H 9850 4800 50  0001 C CNN
 F 1 "GND" H 9850 4900 50  0000 C CNN
 F 2 "" H 9850 5050 50  0000 C CNN
@@
 	10100 5450 10050 5450
 $Comp
-L GND #PWR036
+L GND #PWR035
 U 1 1 5857AA49
 P 10150 5500
-F 0 "#PWR036" H 10150 5250 50  0001 C CNN
+F 0 "#PWR035" H 10150 5250 50  0001 C CNN
 F 1 "GND" H 10150 5350 50  0000 C CNN
 F 2 "" H 10150 5500 50  0000 C CNN
@@
 Connection ~ 10100 5500
 $Comp
-L +5V #PWR037
+L +5V #PWR036
 U 1 1 5857ACB4
 P 9200 6200
-F 0 "#PWR037" H 9200 6050 50  0001 C CNN
+F 0 "#PWR036" H 9200 6050 50  0001 C CNN
 F 1 "+5V" H 9200 6340 50  0000 C CNN
 F 2 "" H 9200 6200 50  0000 C CNN
@@
 $EndComp
 $Comp
-L GND #PWR038
+L GND #PWR037
 U 1 1 5857AEF9
 P 10100 6200
-F 0 "#PWR038" H 10100 5950 50  0001 C CNN
+F 0 "#PWR037" H 10100 5950 50  0001 C CNN
 F 1 "GND" H 10100 6050 50  0000 C CNN
 F 2 "" H 10100 6200 50  0000 C CNN
@@
 	9350 5650 9350 5900
 $Comp
-L GND #PWR039
+L GND #PWR038
 U 1 1 5857B741
 P 7750 6050
-F 0 "#PWR039" H 7750 5800 50  0001 C CNN
+F 0 "#PWR038" H 7750 5800 50  0001 C CNN
 F 1 "GND" H 7750 5900 50  0000 C CNN
 F 2 "" H 7750 6050 50  0000 C CNN
@@
 $EndComp
 $Comp
-L GND #PWR040
+L GND #PWR039
 U 1 1 5857BFA5
 P 10100 4150
-F 0 "#PWR040" H 10100 3900 50  0001 C CNN
+F 0 "#PWR039" H 10100 3900 50  0001 C CNN
 F 1 "GND" H 10100 4000 50  0000 C CNN
 F 2 "" H 10100 4150 50  0000 C CNN
@@
 $EndComp
 $Comp
-L +5V #PWR041
+L +5V #PWR040
 U 1 1 5857CD08
 P 7350 5500
-F 0 "#PWR041" H 7350 5350 50  0001 C CNN
+F 0 "#PWR040" H 7350 5350 50  0001 C CNN
 F 1 "+5V" H 7350 5640 50  0000 C CNN
 F 2 "" H 7350 5500 50  0000 C CNN
@@
 $EndComp
 $Comp
-L +5V #PWR042
+L +5V #PWR041
 U 1 1 585AA589
 P 4900 6600
-F 0 "#PWR042" H 4900 6450 50  0001 C CNN
+F 0 "#PWR041" H 4900 6450 50  0001 C CNN
 F 1 "+5V" H 4900 6740 50  0000 C CNN
 F 2 "" H 4900 6600 50  0000 C CNN
@@
 	4600 7850 4600 7800
 $Comp
-L GND #PWR043
+L GND #PWR042
 U 1 1 585AB07C
 P 4500 7850
-F 0 "#PWR043" H 4500 7600 50  0001 C CNN
+F 0 "#PWR042" H 4500 7600 50  0001 C CNN
 F 1 "GND" H 4500 7700 50  0000 C CNN
 F 2 "" H 4500 7850 50  0000 C CNN
@@
 $EndComp
 $Comp
-L GND #PWR044
+L GND #PWR043
 U 1 1 585AF1DD
 P 6850 5400
-F 0 "#PWR044" H 6850 5150 50  0001 C CNN
+F 0 "#PWR043" H 6850 5150 50  0001 C CNN
 F 1 "GND" H 6850 5250 50  0000 C CNN
 F 2 "" H 6850 5400 50  0000 C CNN
@@
 Wire Notes Line
 	6300 6300 6300 6750
-NoConn ~ 1250 4300
-NoConn ~ 1250 5350
-NoConn ~ 1250 5450
 NoConn ~ 3150 5350
 NoConn ~ 3150 5250
@@
 $EndComp
 $Comp
-L GND #PWR045
+L GND #PWR044
 U 1 1 585D761E
 P 2600 3100
-F 0 "#PWR045" H 2600 2850 50  0001 C CNN
+F 0 "#PWR044" H 2600 2850 50  0001 C CNN
 F 1 "GND" H 2600 2950 50  0000 C CNN
 F 2 "" H 2600 3100 50  0000 C CNN
@@
 	6900 1100 6850 1100
 $Comp
-L GND #PWR046
+L GND #PWR045
 U 1 1 585F45DF
 P 6900 1150
-F 0 "#PWR046" H 6900 900 50  0001 C CNN
+F 0 "#PWR045" H 6900 900 50  0001 C CNN
 F 1 "GND" H 6900 1000 50  0000 C CNN
 F 2 "" H 6900 1150 50  0000 C CNN
@@
 Connection ~ 6900 1100
 $Comp
-L PWR_FLAG #FLG047
+L PWR_FLAG #FLG046
 U 1 1 585F6218
 P 8050 800
-F 0 "#FLG047" H 8050 895 50  0001 C CNN
+F 0 "#FLG046" H 8050 895 50  0001 C CNN
 F 1 "PWR_FLAG" H 8050 980 50  0000 C CNN
 F 2 "" H 8050 800 50  0000 C CNN
@@
 Connection ~ 8050 850
 $Comp
-L PWR_FLAG #FLG048
+L PWR_FLAG #FLG047
 U 1 1 585F73F4
 P 1400 800
-F 0 "#FLG048" H 1400 895 50  0001 C CNN
+F 0 "#FLG047" H 1400 895 50  0001 C CNN
 F 1 "PWR_FLAG" H 1400 980 50  0000 C CNN
 F 2 "" H 1400 800 50  0000 C CNN
@@
 $EndComp
 Connection ~ 1450 800
-NoConn ~ 1250 4600
 Wire Wire Line
 	9650 950  9700 950
@@
 $EndComp
 $Comp
-L GND #PWR049
+L GND #PWR048
 U 1 1 58742CDF
 P 9500 3850
-F 0 "#PWR049" H 9500 3600 50  0001 C CNN
+F 0 "#PWR048" H 9500 3600 50  0001 C CNN
 F 1 "GND" H 9500 3700 50  0000 C CNN
 F 2 "" H 9500 3850 50  0000 C CNN
@@
 $EndComp
 Connection ~ 9500 4150
+NoConn ~ 1250 4300
+NoConn ~ 1250 4600
+NoConn ~ 1250 5350
+NoConn ~ 1250 5450
+$Comp
+L GND #PWR049
+U 1 1 5856C297
+P 1100 6200
+F 0 "#PWR049" H 1100 5950 50  0001 C CNN
+F 1 "GND" H 1100 6050 50  0000 C CNN
+F 2 "" H 1100 6200 50  0000 C CNN
+F 3 "" H 1100 6200 50  0000 C CNN
+	1    1100 6200
+	0    1    1    0
+$EndComp
+Wire Wire Line
+	1200 6300 1250 6300
+Wire Wire Line
+	1100 6200 1250 6200
+Wire Wire Line
+	1250 6100 1200 6100
+Wire Wire Line
+	1200 6100 1200 6300
+Connection ~ 1200 6200
+$Comp
+L ATMEGA328P-A U1
+U 1 1 5856A373
+P 2150 5100
+F 0 "U1" H 1400 6350 50  0000 L BNN
+F 1 "ATMEGA328P-A" H 2550 3700 50  0000 L BNN
+F 2 "Housings_QFP:TQFP-32_7x7mm_Pitch0.8mm" H 2150 5100 50  0001 C CIN
+F 3 "" H 2150 5100 50  0000 C CNN
+	1    2150 5100
+	1    0    0    -1
+$EndComp
 $EndSCHEMATC
