File: SSTdriver.kicad_pcb (KiCad board)
At the start: 4 copper layers, 47.3 x 56 mm, 67 parts, among them P1 CONN_01X05, P2 USB_OTG, P3 CONN_01X04, Q1 Fairchild_BCV27, Q2 QRE1113, Q3 DMG3415U-7, Q4 DMG3415U-7, U1 ATMEGA328P-A, U2 FT231X, U3 LMV358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

Commit message: Fixed a trace clearance by usb interface chip.
Parts:
- C15, C19: footprint Capacitors_SMD:c_elec_8x10 -> Capacitors_SMD:CP_Elec_6.3x5.8
- moved R18 5.11 mm to (106.1, 124.9)
- moved D2 4.55 mm to (104.0, 120.8)
- moved Q3 3.41 mm to (105.3, 129.1)
- moved C9 2.75 mm to (142.5, 130.8)
- moved PWR1 0.79 mm to (115.2, 144.7)
- moved R3 0.74 mm to (139.9, 91.9)
- moved R4 0.63 mm to (136.9, 91.9)
Routing:
- net VCCUSB: track 27.2 -> 23.0 mm
- net Net-(D2-Pad2): track 8.57 -> 12.5 mm
- net GND: track 66.6 -> 69.5 mm, vias 46 -> 45
- net PWRJ: track 81.4 -> 82.9 mm
- net TXD: track 37.6 -> 38.3 mm
- net Net-(R4-Pad2): track 3.74 -> 3.18 mm
Other:
- board text added: "StarSync Trackers Driver v2.1.1"
- board text removed: "StarSync Trackers Controller Driver v2.1.0"

Commit message: 2.2.0
Other:
- rule pad_to_mask_clearance: 0 -> 0.1016
- board text added: "StarSync Trackers Driver v2.2.0"
- board text removed: "StarSync Trackers Driver v2.1.1"
Changed lines of the file:
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@@
-(kicad_pcb (version 4) (host pcbnew 4.0.7-e2-6376~58~ubuntu17.04.1)
+(kicad_pcb (version 20171130) (host pcbnew 5.0.2-bee76a0~70~ubuntu18.04.1)
   (general
-    (links 157)
-    (no_connects 0)
-    (area 99.9998 82.647366 149.655601 145.1062)
     (thickness 1.6)
     (drawings 14)
@@
     (pad_size 5.1054 5.1054)
     (pad_drill 5.1054)
-    (pad_to_mask_clearance 0)
+    (pad_to_mask_clearance 0.1016)
+    (solder_mask_min_width 0.25)
     (aux_axis_origin 0 0)
     (grid_origin 102.235 141.859)
     (visible_elements FFFFFF7F)
     (pcbplotparams
-      (layerselection 0x010fc_80000007)
+      (layerselection 0x010fc_ffffffff)
       (usegerberextensions true)
+      (usegerberattributes false)
+      (usegerberadvancedattributes false)
+      (creategerberjobfile false)
       (excludeedgelayer true)
       (linewidth 0.100000)
@@
       (hpglpennumber 1)
       (hpglpenspeed 20)
-      (hpglpendiameter 15)
-      (hpglpenoverlay 2)
+      (hpglpendiameter 15.000000)
       (psnegative false)
       (psa4output false)
@@
       (drillshape 0)
       (scaleselection 1)
-      (outputdirectory gerbers/))
+      (outputdirectory "gerbers/"))
   )
   (net 0 "")
@@
     (tags "capacitor 0603")
     (attr smd)
-    (fp_text reference C1 (at 2.3622 0.1016 360) (layer F.SilkS)
+    (fp_text reference C1 (at 2.3622 0.1016) (layer F.SilkS)
       (effects (font (size 1.016 1.016) (thickness 0.1016)))
     )
@@
     (tags "capacitor 0603")
     (attr smd)
-    (fp_text reference C2 (at -2.286 0 360) (layer F.SilkS)
+    (fp_text reference C2 (at -2.286 0) (layer F.SilkS)
       (effects (font (size 1.016 1.016) (thickness 0.1016)))
     )
@@
     (tags "capacitor 0603")
     (attr smd)
-    (fp_text reference C6 (at -2.032 -0.254 360) (layer F.SilkS)
+    (fp_text reference C6 (at -2.032 -0.254) (layer F.SilkS)
       (effects (font (size 1.016 1.016) (thickness 0.1016)))
     )
@@
     (tags "capacitor 0603")
     (attr smd)
-    (fp_text reference C7 (at -2.032 0 360) (layer F.SilkS)
+    (fp_text reference C7 (at -2.032 0) (layer F.SilkS)
       (effects (font (size 1.016 1.016) (thickness 0.1016)))
     )
@@
     (tags "capacitor 0603")
     (attr smd)
-    (fp_text reference C9 (at -2.032 0 360) (layer F.SilkS)
+    (fp_text reference C9 (at -2.032 0) (layer F.SilkS)
       (effects (font (size 1.016 1.016) (thickness 0.1016)))
     )
@@
     (tags "capacitor 0603")
     (attr smd)
-    (fp_text reference C11 (at -2.2726 0.381 360) (layer F.SilkS)
+    (fp_text reference C11 (at -2.2726 0.381) (layer F.SilkS)
       (effects (font (size 1.016 1.016) (thickness 0.1016)))
     )
@@
     (tags "capacitor 0603")
     (attr smd)
-    (fp_text reference C12 (at -2.159 0.254 360) (layer F.SilkS)
+    (fp_text reference C12 (at -2.159 0.254) (layer F.SilkS)
       (effects (font (size 1.016 1.016) (thickness 0.1016)))
     )
@@
     (tags "capacitor 0603")
     (attr smd)
-    (fp_text reference C16 (at -2.1844 -0.4572 540) (layer F.SilkS)
+    (fp_text reference C16 (at -2.1844 -0.4572 180) (layer F.SilkS)
       (effects (font (size 1.016 1.016) (thickness 0.1016)))
     )
@@
     (tags SOD-323)
     (attr smd)
-    (fp_text reference D1 (at -2.159 0.127 360) (layer F.SilkS)
+    (fp_text reference D1 (at -2.159 0.127) (layer F.SilkS)
       (effects (font (size 1.016 1.016) (thickness 0.1016)))
     )
@@
     (tags SOD-323)
     (attr smd)
-    (fp_text reference D2 (at -2.159 0 360) (layer F.SilkS)
+    (fp_text reference D2 (at -2.159 0) (layer F.SilkS)
       (effects (font (size 1.016 1.016) (thickness 0.1016)))
     )
@@
     (tags "resistor 0805")
     (attr smd)
-    (fp_text reference FB1 (at -2.286 -0.1524 360) (layer F.SilkS)
+    (fp_text reference FB1 (at -2.286 -0.1524) (layer F.SilkS)
       (effects (font (size 1.016 1.016) (thickness 0.1016)))
     )
@@
     (solder_mask_margin 0.254)
     (clearance 0.254)
-    (fp_text reference P3 (at -1.905 1.016 360) (layer F.SilkS)
+    (fp_text reference P3 (at -1.905 1.016) (layer F.SilkS)
       (effects (font (size 1.016 1.016) (thickness 0.1016)) (justify left bottom))
     )
@@
     (at 145.24228 116.13896 180)
     (attr smd)
-    (fp_text reference Q2 (at -0.00508 2.42316 360) (layer F.SilkS)
+    (fp_text reference Q2 (at -0.00508 2.42316) (layer F.SilkS)
       (effects (font (size 1.016 1.016) (thickness 0.1016)))
     )
@@
     (tags SOT-23)
     (attr smd)
-    (fp_text reference Q4 (at -2.54 0.762 360) (layer F.SilkS)
+    (fp_text reference Q4 (at -2.54 0.762) (layer F.SilkS)
       (effects (font (size 1.016 1.016) (thickness 0.1016)))
     )
@@
     (tags "resistor 0603")
     (attr smd)
-    (fp_text reference R1 (at 2.159 0 360) (layer F.SilkS)
+    (fp_text reference R1 (at 2.159 0) (layer F.SilkS)
       (effects (font (size 1.016 1.016) (thickness 0.1016)))
     )
@@
     (tags "resistor 0603")
     (attr smd)
-    (fp_text reference R2 (at 2.286 0.127 360) (layer F.SilkS)
+    (fp_text reference R2 (at 2.286 0.127) (layer F.SilkS)
       (effects (font (size 1.016 1.016) (thickness 0.1016)))
     )
@@
     (tags "resistor 0603")
     (attr smd)
-    (fp_text reference R5 (at -2.032 0 360) (layer F.SilkS)
+    (fp_text reference R5 (at -2.032 0) (layer F.SilkS)
       (effects (font (size 1.016 1.016) (thickness 0.1016)))
     )
@@
     (tags "resistor 0603")
     (attr smd)
-    (fp_text reference R6 (at -2.032 -0.127 360) (layer F.SilkS)
+    (fp_text reference R6 (at -2.032 -0.127) (layer F.SilkS)
       (effects (font (size 1.016 1.016) (thickness 0.1016)))
     )
@@
     (tags "resistor 0603")
     (attr smd)
-    (fp_text reference R8 (at -1.905 0 360) (layer F.SilkS)
+    (fp_text reference R8 (at -1.905 0) (layer F.SilkS)
       (effects (font (size 1.016 1.016) (thickness 0.1016)))
     )
@@
     (tags "resistor 0603")
     (attr smd)
-    (fp_text reference R9 (at -1.905 0 360) (layer F.SilkS)
+    (fp_text reference R9 (at -1.905 0) (layer F.SilkS)
       (effects (font (size 1.016 1.016) (thickness 0.1016)))
     )
@@
     (tags "resistor 0603")
     (attr smd)
-    (fp_text reference R14 (at -1.905 -0.508 360) (layer F.SilkS)
+    (fp_text reference R14 (at -1.905 -0.508) (layer F.SilkS)
       (effects (font (size 1.016 1.016) (thickness 0.1016)))
     )
@@
     (tags "resistor 0603")
     (attr smd)
-    (fp_text reference R15 (at -2.032 0.508 360) (layer F.SilkS)
+    (fp_text reference R15 (at -2.032 0.508) (layer F.SilkS)
       (effects (font (size 1.016 1.016) (thickness 0.1016)))
     )
@@
     (tags "resistor 0603")
     (attr smd)
-    (fp_text reference R16 (at -2.032 -0.508 360) (layer F.SilkS)
+    (fp_text reference R16 (at -2.032 -0.508) (layer F.SilkS)
       (effects (font (size 1.016 1.016) (thickness 0.1016)))
     )
@@
     (tags "resistor 0603")
     (attr smd)
-    (fp_text reference R17 (at -0.762 2.159 360) (layer F.SilkS)
+    (fp_text reference R17 (at -0.762 2.159) (layer F.SilkS)
       (effects (font (size 1.016 1.016) (thickness 0.1016)))
     )
@@
     (tags "resistor 0603")
     (attr smd)
-    (fp_text reference R24 (at -1.905 0.127 360) (layer F.SilkS)
+    (fp_text reference R24 (at -1.905 0.127) (layer F.SilkS)
       (effects (font (size 1.016 1.016) (thickness 0.1016)))
     )
@@
     (tags "QFN 0.5")
     (attr smd)
-    (fp_text reference U2 (at -3.175 1.778 360) (layer F.SilkS)
+    (fp_text reference U2 (at -3.175 1.778) (layer F.SilkS)
       (effects (font (size 1.016 1.016) (thickness 0.1016)))
     )
@@
     (tags "Crystal Quarz HC49-SD SMD")
     (attr smd)
-    (fp_text reference Y1 (at -6.731 -2.286 360) (layer F.SilkS)
+    (fp_text reference Y1 (at -6.731 -2.286) (layer F.SilkS)
       (effects (font (size 1.016 1.016) (thickness 0.1016)))
     )
@@
     (solder_mask_margin 0.254)
     (clearance 0.254)
-    (fp_text reference P1 (at -1.524 1.016 360) (layer F.SilkS)
+    (fp_text reference P1 (at -1.524 1.016) (layer F.SilkS)
       (effects (font (size 1.016 1.016) (thickness 0.1016)) (justify left bottom))
     )
@@
   (gr_line (start 102.235 85.8266) (end 102.235 141.859) (angle 90) (layer Edge.Cuts) (width 0.15))
   (gr_line (start 149.5806 141.859) (end 149.5806 85.8266) (angle 90) (layer Edge.Cuts) (width 0.15))
-  (gr_text "StarSync Trackers\nDriver v2.1.1" (at 145.5674 126.5682 90) (layer F.SilkS)
+  (gr_text "StarSync Trackers\nDriver v2.2.0" (at 145.5674 126.5682 90) (layer F.SilkS)
     (effects (font (size 1.016 1.016) (thickness 0.1016)))
   )
@@
   (segment (start 126.0468 130.1242) (end 126.0468 128.4224) (width 0.254) (layer Front) (net 4))
   (segment (start 126.0468 128.4224) (end 125.9452 128.3208) (width 0.254) (layer Front) (net 4))
+  (segment (start 128.4986 133.2884) (end 128.4986 134.445602) (width 0.254) (layer Front) (net 4))
+  (segment (start 126.0468 130.8282) (end 126.0468 130.1242) (width 0.254) (layer Front) (net 4))
+  (segment (start 126.0468 134.393802) (end 126.0468 130.8282) (width 0.254) (layer Front) (net 4))
   (segment (start 128.4986 133.2884) (end 128.498599 134.792401) (width 0.254) (layer Front) (net 4))
+  (segment (start 126.445399 134.792401) (end 126.0468 134.393802) (width 0.254) (layer Front) (net 4))
   (segment (start 128.498599 134.792401) (end 126.445399 134.792401) (width 0.254) (layer Front) (net 4))
-  (segment (start 126.0468 130.8282) (end 126.0468 130.1242) (width 0.254) (layer Front) (net 4))
-  (segment (start 126.445399 134.792401) (end 126.0468 134.393802) (width 0.254) (layer Front) (net 4))
-  (segment (start 126.0468 134.393802) (end 126.0468 130.8282) (width 0.254) (layer Front) (net 4))
-  (segment (start 128.4986 133.2884) (end 128.4986 134.445602) (width 0.254) (layer Front) (net 4))
   (segment (start 130.6696 130.2004) (end 130.6696 128.4224) (width 0.254) (layer Front) (net 5))
   (segment (start 130.6696 128.4224) (end 130.7331 128.3589) (width 0.254) (layer Front) (net 5))
